File: SteeringWheel.kicad_pcb (KiCad board)
At the start: 2 copper layers, 22 parts

Commit message: Component Placement Finished
Parts:
- removed H5, H6, H7, H8: MountingHole_Pad, Connector_Wire:SolderWire-6sqmm_1x01_D3.5mm_OD7mm_Relief
- added C1: 100nF, Capacitor_THT:C_Axial_L3.8mm_D2.6mm_P7.50mm_Horizontal, F.Cu at (126.0, 52.0)
- added C2: 100nF, Capacitor_THT:C_Axial_L3.8mm_D2.6mm_P7.50mm_Horizontal, F.Cu at (122.0, 52.0)
- added C3: 100nF, Capacitor_THT:C_Axial_L3.8mm_D2.6mm_P7.50mm_Horizontal, F.Cu at (122.0, 68.0)
- added C4: 100nF, Capacitor_THT:C_Axial_L3.8mm_D2.6mm_P7.50mm_Horizontal, F.Cu at (126.0, 68.0)
- added C5: 100nF, Capacitor_THT:C_Axial_L3.8mm_D2.6mm_P7.50mm_Horizontal, F.Cu at (142.0, 51.8)
- added C6: 100nF, Capacitor_THT:C_Axial_L3.8mm_D2.6mm_P7.50mm_Horizontal, F.Cu at (158.0, 51.8)
- added J1: DT15-08PA, Connector_DTM:TE_DT15-08PA, B.Cu at (141.0, 102.0)
- added R13: 2430, Resistor_THT:R_Axial_DIN0207_L6.3mm_D2.5mm_P10.16mm_Horizontal, F.Cu at (157.8, 108.0)
- added R14: 3830, Resistor_THT:R_Axial_DIN0207_L6.3mm_D2.5mm_P10.16mm_Horizontal, F.Cu at (157.8, 113.0)
- added R15: 6980, Resistor_THT:R_Axial_DIN0207_L6.3mm_D2.5mm_P10.16mm_Horizontal, F.Cu at (157.8, 118.0)
- added R16: 23200, Resistor_THT:R_Axial_DIN0207_L6.3mm_D2.5mm_P10.16mm_Horizontal, F.Cu at (157.8, 123.0)
- added S1: B3F-4055, Button_Switch_THT:SW_B3F-4055, F.Cu at (104.0, 47.0)
- added S4: B3F-4055, Button_Switch_THT:SW_B3F-4055, F.Cu at (178.0, 47.0)
- added S5: B3F-4055, Button_Switch_THT:SW_B3F-4055, F.Cu at (178.0, 63.0)
- added U1: 74HC7014, Package_DIP:DIP-14_W7.62mm, F.Cu at (130.0, 52.0)
- added U3: 74HCT74, Package_DIP:DIP-14_W7.62mm, F.Cu at (146.0, 52.0)
- H1: value MountingHole_Pad -> MountingHole_Pad_MP; footprint Connector_Wire:SolderWire-1sqmm_1x01_D1.4mm_OD2.7mm_Relief -> MountingHole:MountingHole_3.2mm_M3_DIN965_Pad
- H2, H3, H4: value MountingHole_Pad -> MountingHole_Pad_MP; footprint Connector_Wire:SolderWire-6sqmm_1x01_D3.5mm_OD7mm_Relief -> MountingHole:MountingHole_3.2mm_M3_DIN965_Pad
- R1: value 43.2 -> 10k; footprint Resistor_SMD:R_0805_2012Metric -> Resistor_THT:R_Axial_DIN0207_L6.3mm_D2.5mm_P10.16mm_Horizontal
- R10: value 3830 -> 845; footprint Resistor_SMD:R_0805_2012Metric -> Resistor_THT:R_Axial_DIN0207_L6.3mm_D2.5mm_P10.16mm_Horizontal
- R11: value 6980 -> 1180; footprint Resistor_SMD:R_0805_2012Metric -> Resistor_THT:R_Axial_DIN0207_L6.3mm_D2.5mm_P10.16mm_Horizontal
- R12: value 23200 -> 1650; footprint Resistor_SMD:R_0805_2012Metric -> Resistor_THT:R_Axial_DIN0207_L6.3mm_D2.5mm_P10.16mm_Horizontal
- R2: value 143 -> 100k; footprint Resistor_SMD:R_0805_2012Metric -> Resistor_THT:R_Axial_DIN0207_L6.3mm_D2.5mm_P10.16mm_Horizontal
- R3: value 261 -> 10k; footprint Resistor_SMD:R_0805_2012Metric -> Resistor_THT:R_Axial_DIN0207_L6.3mm_D2.5mm_P10.16mm_Horizontal
- R4: value 412 -> 100k; footprint Resistor_SMD:R_0805_2012Metric -> Resistor_THT:R_Axial_DIN0207_L6.3mm_D2.5mm_P10.16mm_Horizontal
- R5: value 604 -> 43.2; footprint Resistor_SMD:R_0805_2012Metric -> Resistor_THT:R_Axial_DIN0207_L6.3mm_D2.5mm_P10.16mm_Horizontal
- R6: value 845 -> 143; footprint Resistor_SMD:R_0805_2012Metric -> Resistor_THT:R_Axial_DIN0207_L6.3mm_D2.5mm_P10.16mm_Horizontal
- R7: value 1180 -> 261; footprint Resistor_SMD:R_0805_2012Metric -> Resistor_THT:R_Axial_DIN0207_L6.3mm_D2.5mm_P10.16mm_Horizontal
- R8: value 1650 -> 412; footprint Resistor_SMD:R_0805_2012Metric -> Resistor_THT:R_Axial_DIN0207_L6.3mm_D2.5mm_P10.16mm_Horizontal
- R9: value 2430 -> 604; footprint Resistor_SMD:R_0805_2012Metric -> Resistor_THT:R_Axial_DIN0207_L6.3mm_D2.5mm_P10.16mm_Horizontal
- S3: value B3F-4055 -> MRK112-A; footprint Button_Switch_THT:SW_B3F-4055 -> MRK112_A (3):SW_MRK112-A
- moved H1 87.8 mm to (178.0, 75.0)
- moved H4 76.4 mm to (178.0, 111.0)
- moved R2 71.8 mm to (118.0, 41.9), turned to -90 degrees
- moved R1 68.3 mm to (114.0, 41.9), turned to -90 degrees
- moved R4 61.9 mm to (118.0, 57.9), turned to -90 degrees
- moved R3 58.3 mm to (114.0, 57.9), turned to -90 degrees
- moved S2 52.7 mm to (104.0, 63.0)
- moved H3 50.0 mm to (104.0, 111.0)
- moved R11 47.2 mm to (157.8, 98.0)
- moved S3 46.8 mm to (141.0, 120.0)
- moved R12 46.5 mm to (157.8, 103.0)
- moved R5 19.6 mm to (124.0, 123.0), turned to 180 degrees
- moved R8 17.8 mm to (124.0, 108.0), turned to 180 degrees
- moved R10 17.7 mm to (124.1, 98.0), turned to 180 degrees
- moved R6 15.4 mm to (124.0, 118.0), turned to 180 degrees
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Connections:
- H1 pad 1: unconnected-(H1-Pad1) -> (no net)
- H2 pad 1: unconnected-(H2-Pad1) -> (no net)
- H3 pad 1: unconnected-(H3-Pad1) -> (no net)
- H4 pad 1: unconnected-(H4-Pad1) -> (no net)
- R1 pad 1: Net-(R1-Pad1) -> +5V
- R1 pad 2: GND -> Net-(C1-Pad1)
- R2 pad 1: Net-(R2-Pad1) -> +5V
- R2 pad 2: GND -> Net-(C2-Pad1)
- R3 pad 1: Net-(R3-Pad1) -> +5V
- R3 pad 2: GND -> Net-(C3-Pad1)
- R4 pad 1: Net-(R4-Pad1) -> +5V
- R4 pad 2: GND -> Net-(C4-Pad1)
- S2 pad 1: Net-(S2-Pad1) -> GND
- S2 pad 2: Net-(S2-Pad1) -> GND
- S2 pad 3: /MCU/Fuel Reset -> Net-(C3-Pad1)
- S2 pad 4: /MCU/Fuel Reset -> Net-(C3-Pad1)
- S3 pad 1: Net-(S3-Pad1) -> Net-(R5-Pad1)
- S3 pad 2: Net-(S3-Pad1) -> Net-(R6-Pad1)
- S3 pad 3: Net-(S3-Pad3) -> Net-(R7-Pad1)
- S3 pad 4: Net-(S3-Pad3) -> Net-(R8-Pad1)
Other:
- board outline added: 92 x 92 mm
- board text added: "For Instructional Use Only."
- board text added: "SOLIDWORKS Educational Product."

Commit message: Rev 1 Prod
Parts:
- removed H3, H4: MountingHole_Pad_MP, MountingHole:MountingHole_3.2mm_M3_DIN965_Pad
- added C7: 100nF, Capacitor_THT:C_Axial_L3.8mm_D2.6mm_P7.50mm_Horizontal, F.Cu at (146.2, 79.5)
- added C8: 100nF, Capacitor_THT:C_Axial_L3.8mm_D2.6mm_P7.50mm_Horizontal, F.Cu at (146.2, 74.5)
- added D1: LED, LED_THT:LED_D3.0mm, F.Cu at (166.0, 58.0)
- added G***: LOGO, LOGO, F.Cu at (115.0, 77.5)
- added J2: Conn_01x01_Pin, Connector_Wire:SolderWire-0.25sqmm_1x01_D0.65mm_OD2mm_Relief, F.Cu at (160.5, 118.6)
- added J3: Conn_01x01_Pin, Connector_Wire:SolderWire-0.25sqmm_1x01_D0.65mm_OD2mm_Relief, F.Cu at (122.5, 119.1)
- added J4: Conn_01x01_Pin, Connector_Wire:SolderWire-0.25sqmm_1x01_D0.65mm_OD2mm_Relief, F.Cu at (118.0, 119.1)
- added J5: Conn_01x01_Pin, Connector_Wire:SolderWire-0.25sqmm_1x01_D0.65mm_OD2mm_Relief, F.Cu at (165.0, 118.6)
- added R17: 330, Resistor_THT:R_Axial_DIN0207_L6.3mm_D2.5mm_P10.16mm_Horizontal, F.Cu at (158.0, 58.0)
- added U2: L7805, Package_TO_SOT_THT:TO-220-3_Horizontal_TabDown, F.Cu at (142.2, 79.5)
- J1: value DT15-08PA -> DTM15-12PA; footprint Connector_DTM:TE_DT15-08PA -> Connector:TE_DTM15-12PA
- moved S3 26.5 mm to (141.0, 93.5)
- moved R16 19.3 mm to (172.8, 111.0)
- moved R11 19.3 mm to (172.9, 86.0)
- moved R12 19.3 mm to (172.9, 91.0)
- moved R13 19.3 mm to (172.9, 96.0)
- moved R14 19.3 mm to (172.9, 101.0)
- moved R15 19.3 mm to (172.9, 106.0)
- moved R10 19.1 mm to (109.2, 86.0)
- moved R5 19.1 mm to (109.2, 111.0)
- moved R6 19.1 mm to (109.2, 106.0)
- moved R7 19.1 mm to (109.2, 101.0)
- moved R8 19.1 mm to (109.2, 96.0)
- moved R9 19.1 mm to (109.2, 91.0)
- moved J1 13.1 mm to (141.0, 115.1), turned to 180 degrees
- moved C3 4.25 mm to (126.2, 68.0)
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Connections:
- J1 pad 1: +5V -> GND
- J1 pad 2: /TCSW -> /Neutral
- J1 pad 3: /MAP2 -> /FuelReset
- J1 pad 4: /MAP1 -> /TCSW
- J1 pad 5: /PitLimit -> /MAP1
- J1 pad 6: /FuelReset -> /MAP2
- J1 pad 7: /Neutral -> /PitLimit
- J1 pad 8: GND -> /DOWNSHIFT
Routing:
- net +5V: track 0.00 -> 168.4 mm
- net /FuelReset: track 0.00 -> 73.9 mm
- net /MAP1: track 0.00 -> 71.7 mm
- net /PitLimit: track 0.00 -> 66.9 mm
- net /MAP2: track 0.00 -> 60.6 mm
- net +12V: track 0.00 -> 56.6 mm
- net /Neutral: track 0.00 -> 56.2 mm
- net Net-(U3B-~{R}): track 0.00 -> 36.9 mm
- net Net-(R5-Pad1): track 0.00 -> 35.1 mm
- net Net-(R16-Pad1): track 0.00 -> 33.1 mm
- net Net-(R11-Pad1): track 0.00 -> 32.9 mm
- net Net-(U3B-C): track 0.00 -> 32.5 mm
- net Net-(R6-Pad1): track 0.00 -> 31.9 mm
- net Net-(R15-Pad1): track 0.00 -> 31.6 mm
- net Net-(R13-Pad1): track 0.00 -> 30.5 mm
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- added copper zone on B.Cu, net GND
- added copper zone on F.Cu, net GND
Other:
- board text added: "00"
- board text added: "01"
- board text added: "02"
- board text added: "03"
- board text added: "04"
- board text added: "05"
- board text added: "06"
- board text added: "07"
- board text added: "08"
- board text added: "09"
- board text added: "1"
- board text added: "10"
- board text added: "11"
- board text added: "12"
- board text added: "FUEL RESET"
- board text added: "MAP"
- board text added: "NEUTRAL"
- board text added: "ON"
- board text added: "PIT LIMIT"
