File: SteeringWheel.kicad_sch (KiCad schematic)
At the start: 0 parts

Commit message: Component Placement Finished
Parts:
- added C1, C2, C3, C4, C5, C6: 100nF, Capacitor_THT:C_Axial_L3.8mm_D2.6mm_P7.50mm_Horizontal, symbol Device:C
- added H1, H2, H3, H4: MountingHole_Pad_MP, MountingHole:MountingHole_3.2mm_M3_DIN965_Pad, symbol Mechanical:MountingHole_Pad_MP
- added J1: DT15-08PA, Connector_DTM:TE_DT15-08PA, symbol DT15-08PA:DT15-08PA
- added R1, R3: 10k, Resistor_THT:R_Axial_DIN0207_L6.3mm_D2.5mm_P10.16mm_Horizontal, symbol Device:R
- added R10: 845, Resistor_THT:R_Axial_DIN0207_L6.3mm_D2.5mm_P10.16mm_Horizontal, symbol Device:R
- added R11: 1180, Resistor_THT:R_Axial_DIN0207_L6.3mm_D2.5mm_P10.16mm_Horizontal, symbol Device:R
- added R12: 1650, Resistor_THT:R_Axial_DIN0207_L6.3mm_D2.5mm_P10.16mm_Horizontal, symbol Device:R
- added R13: 2430, Resistor_THT:R_Axial_DIN0207_L6.3mm_D2.5mm_P10.16mm_Horizontal, symbol Device:R
- added R14: 3830, Resistor_THT:R_Axial_DIN0207_L6.3mm_D2.5mm_P10.16mm_Horizontal, symbol Device:R
- added R15: 6980, Resistor_THT:R_Axial_DIN0207_L6.3mm_D2.5mm_P10.16mm_Horizontal, symbol Device:R
- added R16: 23200, Resistor_THT:R_Axial_DIN0207_L6.3mm_D2.5mm_P10.16mm_Horizontal, symbol Device:R
- added R2, R4: 100k, Resistor_THT:R_Axial_DIN0207_L6.3mm_D2.5mm_P10.16mm_Horizontal, symbol Device:R
- added R5: 43.2, Resistor_THT:R_Axial_DIN0207_L6.3mm_D2.5mm_P10.16mm_Horizontal, symbol Device:R
- added R6: 143, Resistor_THT:R_Axial_DIN0207_L6.3mm_D2.5mm_P10.16mm_Horizontal, symbol Device:R
- added R7: 261, Resistor_THT:R_Axial_DIN0207_L6.3mm_D2.5mm_P10.16mm_Horizontal, symbol Device:R
- added R8: 412, Resistor_THT:R_Axial_DIN0207_L6.3mm_D2.5mm_P10.16mm_Horizontal, symbol Device:R
- added R9: 604, Resistor_THT:R_Axial_DIN0207_L6.3mm_D2.5mm_P10.16mm_Horizontal, symbol Device:R
- added S1, S2, S4, S5: B3F-4055, Button_Switch_THT:SW_B3F-4055, symbol B3F-4055:B3F-4055
- added S3: MRK112-A, MRK112_A (3):SW_MRK112-A, symbol MRK112-A:MRK112-A
- added U1: 74HC7014, Package_DIP:DIP-14_W7.62mm, symbol 74xx:74HC7014
- added U3: 74HCT74, Package_DIP:DIP-14_W7.62mm, symbol 74xx:74HCT74
Connections:
- new net: C2.1, R2.2, U1.3
- new net: U1.4, U3.1 (~{R})
- new net: R15.1, S3.11
- new net: C1.1, R1.2, S1.3, S1.4, U1.1
- new net: U1.2, U3.3 (C)
- new net: R16.1, S3.12
- new net: R8.1, S3.4
- new net: R14.1, S3.10
- new net: C4.1, R4.2, U1.9
- new net: R13.1, S3.9
- new net: C3.1, R3.2, S2.3, S2.4, U1.5
- new net: R9.1, S3.5
- new net: U3.2 (D), U3.6 (~{Q})
- new net: U1.8, U3.13 (~{R})
- new net: R5.1, S3.1
- new net: R10.1, S3.6
- new net: U1.6, U3.11 (C)
- new net: R12.1, S3.8
- new net: R6.1, S3.2
- new net: R7.1, S3.3
- new net: R11.1, S3.7
- new net +5V: C5.1, C6.1, J1.1, R1.1, R2.1, R3.1, R4.1, S4.1, S4.2, U1.14 (VCC), U3.10 (~{S}), U3.14 (VCC), U3.4 (~{S})
- new net FuelReset: J1.6, S4.3, S4.4
- new net GND: C1.2, C2.2, C3.2, C4.2, C5.2, C6.2, J1.8, R10.2, R11.2, R12.2, R13.2, R14.2, R15.2, R16.2, R5.2, R6.2, R7.2, R8.2, R9.2, S1.1, S1.2, S2.1, S2.2, S5.1, S5.2, U1.7 (GND), U3.7 (GND)
- new net MAP1: J1.4, U3.12 (D), U3.8 (~{Q})
- new net MAP2: J1.3, U3.9 (Q)
- new net Neutral: J1.7, S5.3, S5.4
- new net PitLimit: J1.5, U3.5 (Q)
- new net TCSW: J1.2, S3.A
Other:
- removed sheet MCU
- company: (none) -> Owls Racing
- title: (none) -> Steering Wheel

Commit message: Rev 1 Prod
Parts:
- removed H3, H4: MountingHole_Pad_MP, MountingHole:MountingHole_3.2mm_M3_DIN965_Pad, symbol Mechanical:MountingHole_Pad_MP
- removed J1: DT15-08PA, Connector_DTM:TE_DT15-08PA, symbol DT15-08PA:DT15-08PA
- added C7, C8: 100nF, Capacitor_THT:C_Axial_L3.8mm_D2.6mm_P7.50mm_Horizontal, symbol Device:C
- added D1: LED, LED_THT:LED_D3.0mm, symbol Device:LED
- added J1: DTM15-12PA, Connector:TE_DTM15-12PA, symbol DTM15-12PA:DTM15-12PA
- added J2, J3, J4, J5: Conn_01x01_Pin, Connector_Wire:SolderWire-0.25sqmm_1x01_D0.65mm_OD2mm_Relief, symbol Connector:Conn_01x01_Pin
- added R17: 330, Resistor_THT:R_Axial_DIN0207_L6.3mm_D2.5mm_P10.16mm_Horizontal, symbol Device:R
- added U2: L7805, Package_TO_SOT_THT:TO-220-3_Horizontal_TabDown, symbol Regulator_Linear:L7805
Connections:
- net +5V: now also C8.1, R17.2, U2.3 (OUT)
- net FuelReset: now also J1.3
- net GND: now also C7.2, C8.2, D1.1 (K), J1.1, J4.1 (Pin_1), J5.1 (Pin_1), U2.2 (GND)
- net MAP1: now also J1.5
- net MAP2: now also J1.6
- net Neutral: now also J1.2
- net PitLimit: now also J1.7
- net TCSW: now also J1.4
- new net: D1.2 (A), R17.1
- new net +12V: C7.1, J1.12, U2.1 (IN)
- new net DOWNSHIFT: J1.8, J3.1 (Pin_1)
- new net UPSHIFT: J1.11, J2.1 (Pin_1)
